File: ESP32-Drone.kicad_sch (KiCad schematic)
At the start: 7 parts

Commit message: Test branching 1
Other:
- sheet ESP32 ports: added USB_DN, USB_DP; removed none
- sheet Power Management ports: added USB_DN, USB_DP; removed none
Changed lines of the file:
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@@
+		)
+	)
+	(wire
+		(pts
+			(xy 160.02 220.98) (xy 187.96 220.98)
+		)
+		(stroke
+			(width 0)
+			(type default)
 		)
 	)
@@
 		(pts
 			(xy 356.87 55.88) (xy 356.87 57.15)
+		)
+		(stroke
+			(width 0)
+			(type default)
+		)
+	)
+	(wire
+		(pts
+			(xy 160.02 227.33) (xy 187.96 227.33)
 		)
 		(stroke
@@
 			)
 		)
+		(pin "USB_DN" bidirectional
+			(at 160.02 227.33 0)
+			(effects
+				(font
+					(size 1.27 1.27)
+				)
+				(justify right)
+			)
+		)
+		(pin "USB_DP" bidirectional
+			(at 160.02 220.98 0)
+			(effects
+				(font
+					(size 1.27 1.27)
+				)
+				(justify right)
+			)
+		)
 		(instances
 			(project "ESP32-Drone"
@@
 			)
 		)
+		(pin "USB_DN" bidirectional
+			(at 187.96 227.33 180)
+			(effects
+				(font
+					(size 1.27 1.27)
+				)
+				(justify left)
+			)
+		)
+		(pin "USB_DP" bidirectional
+			(at 187.96 220.98 180)
+			(effects
+				(font
+					(size 1.27 1.27)
+				)
+				(justify left)
+			)
+		)
