File: ESP32-Drone.kicad_sch (KiCad schematic)
At the start: 7 parts

Commit message: First commit test with library test
Parts:
- added U6: CD4013BE, digikey-footprints:DIP-14_W3mm, symbol Digikey_flip_flops:CD4013BE
Changed lines of the file:
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@@
+	)
+	(symbol
+		(lib_id "Digikey_flip_flops:CD4013BE")
+		(at 44.45 217.17 0)
+		(unit 1)
+		(exclude_from_sim no)
+		(in_bom yes)
+		(on_board yes)
+		(dnp no)
+		(fields_autoplaced yes)
+		(property "Reference" "U6"
+			(at 49.1333 209.55 0)
+			(effects
+				(font
+					(size 1.524 1.524)
+				)
+				(justify left)
+			)
+		)
+		(property "Value" "CD4013BE"
+			(at 49.1333 212.09 0)
+			(effects
+				(font
+					(size 1.524 1.524)
+				)
+				(justify left)
+			)
+		)
+		(property "Footprint" "digikey-footprints:DIP-14_W3mm"
+			(at 49.53 212.09 0)
+			(effects
+				(font
+					(size 1.524 1.524)
+				)
+				(justify left)
+				(hide yes)
+			)
+		)
+		(property "Datasheet" "http://www.ti.com/general/docs/suppproductinfo.tsp?distId=10&gotoUrl=http%3A%2F%2Fwww.ti.com%2Flit%2Fgpn%2Fcd4013b"
+			(at 49.53 209.55 0)
+			(effects
+				(font
+					(size 1.524 1.524)
+				)
+				(justify left)
+				(hide yes)
+			)
+		)
+		(property "Description" "IC FF D-TYPE DUAL 1BIT 14DIP"
+			(at 44.45 217.17 0)
+			(effects
+				(font
+					(size 1.27 1.27)
+				)
+				(hide yes)
+			)
+		)
+		(property "Digi-Key_PN" "296-2033-5-ND"
+			(at 49.53 207.01 0)
+			(effects
+				(font
+					(size 1.524 1.524)
+				)
+				(justify left)
+				(hide yes)
+			)
+		)
+		(property "MPN" "CD4013BE"
+			(at 49.53 204.47 0)
+			(effects
+				(font
+					(size 1.524 1.524)
+				)
+				(justify left)
+				(hide yes)
+			)
+		)
+		(property "Category" "Integrated Circuits (ICs)"
+			(at 49.53 201.93 0)
+			(effects
+				(font
+					(size 1.524 1.524)
+				)
+				(justify left)
+				(hide yes)
+			)
+		)
+		(property "Family" "Logic - Flip Flops"
+			(at 49.53 199.39 0)
+			(effects
+				(font
+					(size 1.524 1.524)
+				)
+				(justify left)
+				(hide yes)
+			)
+		)
+		(property "DK_Datasheet_Link" "http://www.ti.com/general/docs/suppproductinfo.tsp?distId=10&gotoUrl=http%3A%2F%2Fwww.ti.com%2Flit%2Fgpn%2Fcd4013b"
+			(at 49.53 196.85 0)
+			(effects
+				(font
+					(size 1.524 1.524)
+				)
+				(justify left)
+				(hide yes)
+			)
+		)
+		(property "DK_Detail_Page" "/product-detail/en/texas-instruments/CD4013BE/296-2033-5-ND/67245"
+			(at 49.53 194.31 0)
+			(effects
+				(font
+					(size 1.524 1.524)
+				)
+				(justify left)
+				(hide yes)
+			)
+		)
+		(property "Description_1" "IC FF D-TYPE DUAL 1BIT 14DIP"
+			(at 49.53 191.77 0)
+			(effects
+				(font
+					(size 1.524 1.524)
+				)
+				(justify left)
+				(hide yes)
+			)
+		)
+		(property "Manufacturer" "Texas Instruments"
+			(at 49.53 189.23 0)
+			(effects
+				(font
+					(size 1.524 1.524)
+				)
+				(justify left)
+				(hide yes)
+			)
+		)
+		(property "Status" "Active"
+			(at 49.53 186.69 0)
+			(effects
+				(font
+					(size 1.524 1.524)
+				)
+				(justify left)
+				(hide yes)
+			)
+		)
+		(pin "5"
+		)
+		(pin "7"
+		)
+		(pin "4"
+		)
+		(pin "8"
+		)
+		(pin "9"
+		)
+		(pin "10"
+		)
+		(pin "14"
+		)
+		(pin "3"
+		)
+		(pin "6"
+		)
+		(pin "11"
+		)
+		(pin "12"
+		)
+		(pin "2"
+		)
+		(pin "13"
+		)
+		(pin "1"
+		)
+		(instances
+			(project ""
+				(path "/3c0e038e-28f7-4e96-beb4-6e0ecd959d7c"
+					(reference "U6")
+					(unit 1)
+				)
+			)
+		)
 	)
 	(symbol

Commit message: I added a flip flop for digikey library test
Parts:
- U6: footprint digikey-footprints:DIP-14_W3mm -> Digikey_Footprints:SOIC-14_W3.9mm
Changed lines of the file:
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@@
 			)
 		)
-		(property "Footprint" "digikey-footprints:DIP-14_W3mm"
+		(property "Footprint" "Digikey_Footprints:SOIC-14_W3.9mm"
 			(at 49.53 212.09 0)
 			(effects
