File: Power-Management.kicad_sch (KiCad schematic)
At the start: 0 parts

Commit message: Test branching 1
Parts:
- added C1, C3: 10μF, symbol Device:C
- added C2: 2.2μF, symbol Device:C
- added D1: SS34, Diode_SMD:D_SMA, symbol Diode:SS34
- added D2, D3, D4: LED, symbol Device:LED
- added J1: USB_C_Receptacle_USB2.0_16P, Connector_USB:USB_C_Receptacle_HCTL_HC-TYPE-C-16P-01A, symbol AI_CONNECTORS:USB_C_Receptacle_USB2.0_16P
- added J2: B2B-PH-SM4-TB, AI_CONNECTORS:B2B-PH-SM4-TB, symbol AI_CONNECTORS:B2B-PH-SM4-TB_LF__SN_
- added Q1: Q_PMOS_GSD, symbol Transistor_FET:Q_PMOS_GSD
- added R1: 100K, Resistor_SMD:R_0603_1608Metric, symbol AI_RESISTORS:100K_SMD_Resistor
- added R10, R9: 100K, symbol Device:R
- added R2, R3: 5K1, Resistor_SMD:R_0603_1608Metric, symbol AI_RESISTORS:5K1 Resistor
- added R4: 470R, Resistor_SMD:R_0603_1608Metric, symbol Device:R
- added R5: 3K3, symbol Device:R
- added R6, R8: 1K3, Resistor_SMD:R_0603_1608Metric, symbol Device:R
- added R7: 100K, Resistor_SMD:R_0603_1608Metric, symbol Device:R
- added SW2: SW_SPDT, symbol Switch:SW_SPDT
- added U2: MIC5219-3.3YM5, Package_TO_SOT_SMD:SOT-23-5, symbol Regulator_Linear:MIC5219-3.3YM5
- added U3: TP4056, TP4056:SOP127P600X175-9N, symbol AI_IC:TP4056
Connections:
- new net: R7.2, SW2.1 (A)
- new net: D4.1 (K), R8.2
- new net: D3.1 (K), R6.2
- new net: D2.2 (A), R4.2
- new net: R5.1, U3.2 (PROG)
- new net +3V3: C2.1, C3.1, R4.1, U2.5 (OUT)
- new net +5V: D1.2 (A), J1.A4 (VBUS), J1.A9 (VBUS), J1.B4 (VBUS), J1.B9 (VBUS), Q1.1 (G), R1.1
- new net +VBatt: J2.2, Q1.3 (D), U3.5 (BAT)
- new net +Vbus: C1.1, D1.1 (K), D3.2 (A), D4.2 (A), Q1.2 (S), R7.1, R9.1, U2.1 (IN), U3.4 (VCC), U3.8 (CE)
- new net BATT_Vdc: R10.1, R9.2
- new net CC1: J1.A5 (CC1), R2.1
- new net CC2: J1.B5 (CC2), R3.1
- new net CHRG: R6.1, U3.7 (~{CHRG})
- new net GND: C1.2, C2.2, C3.2, D2.1 (K), J1.A1 (GND), J1.A12 (GND), J1.B1 (GND), J1.B12 (GND), J1.S1 (SHIELD), J2.1, R1.2, R10.2, R2.2, R3.2, R5.2, SW2.3 (C), U2.2 (GND), U3.1 (TEMP), U3.3 (GND), U3.9 (EP)
- new net LDO_EN: SW2.2 (B), U2.3 (EN)
- new net STDBY: R8.1, U3.6 (~{STDBY})
- new net USB_DN: J1.A7 (D-), J1.B7 (D-)
- new net USB_DP: J1.A6 (D+), J1.B6 (D+)
- no-connect marks 0 -> 3
Other:
- note added: "Battery Voltage Measurement"
- note added: "USB Input for charging LiPo batt"
- note added: "Vbatt (max) = 4.2V Vbatt (min) = 3.2V Adc Pin Voltage = 1.5V to 2.1V"
