File: Peripherals.kicad_sch (KiCad schematic)
At the start: 0 parts

Commit message: All component assembly ready. Pending net classifications
Parts:
- added C11: 10μF, Capacitor_SMD:C_0603_1608Metric, symbol AI_CAPACITORS:C
- added C12, C13: 100nF, Capacitor_SMD:C_0603_1608Metric, symbol AI_CAPACITORS:C
- added C14, C15, C16, C17: 22μF, Capacitor_SMD:C_0603_1608Metric, symbol AI_CAPACITORS:C
- added D10, D11, D5, D9: 1N4148WS, Diode_SMD:D_SOD-323, symbol Diode:1N4148WS
- added D6, D7, D8: LED, symbol Device:LED
- added J5, J6, J7, J8: Conn_01x02, Connector_PinHeader_2.54mm:PinHeader_1x02_P2.54mm_Vertical, symbol AI_CONNECTORS:Conn_01x02
- added Q3, Q4, Q5, Q6: Si2302CDS-T1-GE3, Package_TO_SOT_SMD:SOT-23, symbol AI_MOSFETS:Si2302CDS-T1-GE3
- added R16: 5K1, Resistor_SMD:R_0603_1608Metric, symbol AI_RESISTORS:R
- added R17, R18, R19, R23, R24, R25: 10K, Resistor_SMD:R_0603_1608Metric, symbol AI_RESISTORS:R
- added R20, R21, R22: 1K3, Resistor_SMD:R_0603_1608Metric, symbol AI_RESISTORS:R
- added U5: MPU-6050, Sensor_Motion:InvenSense_QFN-24_4x4mm_P0.5mm, symbol Sensor_Motion:MPU-6050
Connections:
- new net: C14.2, D5.2 (A), J5.2 (Pin_2), Q3.3 (D)
- new net: D8.2 (A), R22.2
- new net: C15.2, D9.2 (A), J6.2 (Pin_2), Q4.3 (D)
- new net: D7.2 (A), R21.2
- new net: C13.1, U5.20 (CPOUT)
- new net: C16.2, D10.2 (A), J7.2 (Pin_2), Q5.3 (D)
- new net: R16.1, U5.9 (AD0)
- new net: C17.2, D11.2 (A), J8.2 (Pin_2), Q6.3 (D)
- new net: D6.2 (A), R20.2
- new net: C12.1, U5.10 (REGOUT)
- new net +3V3: C11.1, R17.1, R18.1, U5.13 (VDD), U5.8 (VLOGIC)
- new net +VBatt: C14.1, C15.1, C16.1, C17.1, D10.1 (K), D11.1 (K), D5.1 (K), D9.1 (K), J5.1 (Pin_1), J6.1 (Pin_1), J7.1 (Pin_1), J8.1 (Pin_1)
- new net GND: C11.2, C12.2, C13.2, D6.1 (K), D7.1 (K), D8.1 (K), Q3.2 (S), Q4.2 (S), Q5.2 (S), Q6.2 (S), R16.2, R19.2, R23.2, R24.2, R25.2, U5.1 (CLKIN), U5.11 (FSYNC), U5.18 (GND)
- new net LED_1: R20.1
- new net LED_2: R21.1
- new net LED_3: R22.1
- new net MOTOR_1: Q3.1 (G), R19.1
- new net MOTOR_2: Q4.1 (G), R23.1
- new net MOTOR_3: Q5.1 (G), R24.1
- new net MOTOR_4: Q6.1 (G), R25.1
- new net SCL: R17.2, U5.23 (SCL)
- new net SDA: R18.2, U5.24 (SDA)
- new net SRV2: U5.12 (INT)
- no-connect marks 0 -> 2
